File: cargador-cargador/cargador-cargador.kicad_sch (KiCad schematic)
At the start: 7 parts, among them J1 Jack DC, J2 salida, U1 L7805

Commit message: little responsive
Parts:
- D1: footprint LED_SMD:LED_0603_1608Metric_Pad1.05x0.95mm_HandSolder -> EESTN5:Pin_strip_2
- R1: footprint EESTN5:R_1206 -> EESTN5:RES0.3
Changed lines of the file:
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@@
       (effects (font (size 1.27 1.27)) (justify left))
     )
-    (property "Footprint" "EESTN5:R_1206" (at 99.06 44.45 0)
+    (property "Footprint" "EESTN5:RES0.3" (at 99.06 44.45 0)
       (effects (font (size 1.524 1.524)) hide)
     )
@@
       (effects (font (size 1.27 1.27)) (justify right))
     )
-    (property "Footprint" "LED_SMD:LED_0603_1608Metric_Pad1.05x0.95mm_HandSolder" (at 99.06 52.07 0)
+    (property "Footprint" "EESTN5:Pin_strip_2" (at 99.06 52.07 0)
       (effects (font (size 1.27 1.27)) hide)
     )
