File: cargador-cargador/cargador-cargador.kicad_pcb (KiCad board)
At the start: 2 copper layers, 15 x 20 mm, 7 parts, among them J1 Jack DC, J2 salida, U1 L7805

Commit message: little responsive
Parts:
- added hole_2mm: VAL**, EESTN5:hole_2mm, F.Cu at (78.3, 41.8)
- added hole_2mm: VAL**, EESTN5:hole_2mm, F.Cu at (61.8, 58.2)
- D1: footprint LED_SMD:LED_0603_1608Metric_Pad1.05x0.95mm_HandSolder -> EESTN5:Pin_strip_2
- R1: footprint EESTN5:R_1206 -> EESTN5:RES0.3
- moved J2 8.08 mm to (78.5, 47.5)
- moved D1 6.02 mm to (73.7, 48.9)
- moved R2 5.82 mm to (78.5, 54.1)
- moved R1 4.94 mm to (69.3, 52.5), turned to 0 degrees
- moved U1 4.10 mm to (69.6, 56.7)
- moved C1 1.48 mm to (73.5, 43.7)
- moved J1 0.44 mm to (68.0, 44.6)
Routing:
- net Net-(D1-K): track 14.3 -> 23.0 mm
- net Net-(U1-OUT): track 16.4 -> 20.0 mm
- net Net-(U1-IN): track 22.3 -> 19.3 mm
- net Net-(D1-A): track 2.13 -> 3.90 mm
- net GND: track 20.5 -> 21.7 mm
Other:
- board size 15 x 20 mm -> 20 x 20 mm

Commit message: rework
Routing:
- net GND: track 21.7 -> 0.06 mm
- added copper zone on B.Cu, net GND
Changed lines of the file:
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@@
     (pad_to_mask_clearance 0)
     (pcbplotparams
-      (layerselection 0x00010fc_ffffffff)
+      (layerselection 0x0000000_fffffffe)
       (plot_on_all_layers_selection 0x0000000_00000000)
       (disableapertmacros false)
@@
       (sketchpadsonfab false)
       (subtractmaskfromsilk false)
-      (outputformat 1)
+      (outputformat 5)
       (mirror false)
-      (drillshape 1)
+      (drillshape 2)
       (scaleselection 1)
       (outputdirectory "")
@@
   (segment (start 73.5 44.7) (end 68.14 44.7) (width 1) (layer "B.Cu") (net 1))
   (segment (start 68.14 44.7) (end 68.04 44.6) (width 1) (layer "B.Cu") (net 1))
-  (segment (start 66.2 40.7) (end 72.8 40.7) (width 1) (layer "B.Cu") (net 2))
-  (segment (start 64.8 45.3) (end 64.8 42.1) (width 1) (layer "B.Cu") (net 2))
-  (segment (start 72.8 40.7) (end 73.5 41.4) (width 1) (layer "B.Cu") (net 2))
-  (segment (start 61.84 44.6) (end 64.8 44.6) (width 1) (layer "B.Cu") (net 2))
   (segment (start 64.8 49.26) (end 64.84 49.3) (width 1) (layer "B.Cu") (net 2))
-  (segment (start 73.5 41.4) (end 73.5 42.7) (width 1) (layer "B.Cu") (net 2))
-  (segment (start 64.8 45.3) (end 64.8 49.26) (width 1) (layer "B.Cu") (net 2))
-  (segment (start 64.8 42.1) (end 66.2 40.7) (width 1) (layer "B.Cu") (net 2))
-  (segment (start 64.8 44.6) (end 64.8 45.3) (width 1) (layer "B.Cu") (net 2))
   (segment (start 69.6 57.75) (end 70.3 58.45) (width 0.75) (layer "B.Cu") (net 3))
   (segment (start 74.97 48.9) (end 78.5 48.9) (width 1) (layer "B.Cu") (net 3))
@@
   (segment (start 67.06 56.7) (end 67.06 58.76) (width 0.75) (layer "B.Cu") (net 5))
   (segment (start 74.6 59.5) (end 76.19 57.91) (width 0.75) (layer "B.Cu") (net 5))
+  (zone (net 2) (net_name "GND") (layer "B.Cu") (hatch edge 0.5)
+    (connect_pads (clearance 0.75))
+    (min_thickness 1) (filled_areas_thickness no)
+    (fill yes (thermal_gap 0.75) (thermal_bridge_width 1))
+    (polygon
+      (pts
+        (xy 60 40)
+        (xy 80 40)
+        (xy 80 60)
+        (xy 60 60)
+      )
+    )
+  )
 )
