File: LightNing 3.0.kicad_pcb (KiCad board)
At the start: 2 copper layers, 50 x 50 mm, 35 parts, among them J1 Motor_Izq_B, J2 Motor_Der_A, J3 Motor_Izq_A, J4 Motor_Der_B, J5 Jack DC, J6 batt, J7 salida esp-usb, J8 LED_izq, J9 LED_izq, SW1 SW_SPDT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

Commit message: uno cambio lokos
Parts:
- removed C2: 100uF 25v, EESTN5:CAP_ELEC_SMD_4X5.5
- removed J3: Motor_Izq_A, EESTN5:BORNERA2_AZUL
- removed J5: Jack DC, Connector_BarrelJack:BarrelJack_Kycon_KLDX-0202-xC_Horizontal
- removed J7: salida esp-usb, EESTN5:Pin_Header_5
- removed R2: 22 2W, EESTN5:RES0.3
- removed U2: L7805, EESTN5:TO-220
- added hole_2mm: VAL**, EESTN5:hole_2mm, F.Cu at (43.0, 24.0)
- added hole_2mm: VAL**, EESTN5:hole_2mm, F.Cu at (92.0, 68.0)
- added hole_2mm: VAL**, EESTN5:hole_2mm, F.Cu at (43.0, 68.0)
- C1, C3, C4: footprint EESTN5:CAP_ELEC_SMD_4X5.5 -> EESTN5:CAP_ELEC_5x11mm
- C5, C6, D1, D2, D3, D4, D5, D6, D7, D8: moved to B.Cu
- D9: footprint LED_SMD:LED_0603_1608Metric_Pad1.05x0.95mm_HandSolder -> EESTN5:LED_1206
- J1: value Motor_Izq_B -> motores izq; footprint EESTN5:BORNERA2_AZUL -> EESTN5:JST-4V
- J2: value Motor_Der_A -> motores der; footprint EESTN5:BORNERA2_AZUL -> EESTN5:JST-4V
- J4: value Motor_Der_B -> esp32 usb y batt; footprint EESTN5:BORNERA2_AZUL -> EESTN5:Pin_Header_6
- J8, J9: footprint EESTN5:JST-3V -> EESTN5:Pin_Strip_3
- R1: value 330 -> 220
- moved D7 156.8 mm to (60.4, 32.0), turned to 180 degrees
- moved D8 153.4 mm to (65.1, 32.0), turned to 180 degrees
- moved D5 149.7 mm to (60.4, 37.7), turned to 180 degrees
- moved D3 149.6 mm to (60.4, 35.8), turned to 180 degrees
- moved D1 149.3 mm to (60.4, 33.9), turned to 180 degrees
- moved D6 146.2 mm to (65.1, 37.7), turned to 180 degrees
- moved D4 146.1 mm to (65.1, 35.8), turned to 180 degrees
- moved D2 145.7 mm to (65.1, 33.9), turned to 180 degrees
- moved U1 136.4 mm to (83.0, 51.5), turned to 90 degrees
- moved C5 135.9 mm to (64.5, 58.3)
- moved C4 135.8 mm to (51.8, 61.1), turned to 180 degrees
- moved SW1 134.9 mm to (44.6, 47.6)
- moved D9 133.5 mm to (74.0, 56.7), turned to 90 degrees
- moved C6 132.7 mm to (58.6, 58.3), turned to 180 degrees
- moved J2 130.3 mm to (89.4, 28.3), turned to 180 degrees
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Connections:
- J1 pad 1: Net-(D3-A) -> Net-(D7-A)
- J2 pad 1: Net-(D5-A) -> Net-(D3-A)
- J2 pad 2: Net-(D7-A) -> Net-(D5-A)
- J4 pad 1: Net-(D7-A) -> /salida
- J4 pad 2: Net-(D5-A) -> +3.3V
- J8 pad 1: +3.3V -> +5V
- J9 pad 1: +3.3V -> +5V
- R1 pad 1: Net-(U2-OUT) -> Net-(D9-K)
- R1 pad 2: Net-(D9-A) -> GND
- SW1 pad 1: Net-(D9-K) -> /salida
- U1 pad 10: /IN3 -> /IN4
- U1 pad 12: /IN4 -> /IN3
- U1 pad 5: /IN1 -> /IN2
- U1 pad 7: /IN2 -> /IN1
- U4 pad 10: /Led_Izq -> unconnected-(U4-DAC_1/ADC2_CH8/GPIO25-Pad10)
- U4 pad 11: /Led_Der -> unconnected-(U4-DAC_2/ADC2_CH9/GPIO26-Pad11)
- U4 pad 24: unconnected-(U4-ADC2_CH2/GPIO2-Pad24) -> Net-(D9-A)
- U4 pad 27: unconnected-(U4-GPIO16-Pad27) -> /Led_Izq
- U4 pad 28: unconnected-(U4-GPIO17-Pad28) -> /Led_Der
Routing:
- net VCC: track 0.00 -> 129.7 mm
- net +5V: track 0.00 -> 109.8 mm, vias 0 -> 2
- net Net-(D5-A): track 0.00 -> 76.5 mm
- net Net-(D3-A): track 0.00 -> 73.5 mm
- net +3.3V: track 0.00 -> 48.0 mm, vias 0 -> 1
- net Net-(D1-A): track 0.00 -> 45.7 mm
- net /TX: track 0.00 -> 40.1 mm, vias 0 -> 1
- net Net-(D7-A): track 0.00 -> 35.8 mm
- net /EN: track 0.00 -> 27.5 mm, vias 0 -> 1
- net /IN4: track 0.00 -> 26.3 mm
- net /Led_Der: track 0.00 -> 25.6 mm, vias 0 -> 1
- net /IN3: track 0.00 -> 23.3 mm
- net /RX: track 0.00 -> 22.9 mm, vias 0 -> 1
- net /salida: track 0.00 -> 20.7 mm
- net /Led_Izq: track 0.00 -> 16.9 mm, vias 0 -> 1
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- added copper zone on B.Cu, net GND
- added copper zone on F.Cu, net GND
Other:
- board size 50 x 50 mm -> 55 x 48 mm

Commit message: a
Parts:
- moved C1 22.3 mm to (86.8, 66.8), turned to 180 degrees
Routing:
- net VCC: track 129.7 -> 134.0 mm
- net +5V: track 109.8 -> 108.5 mm, vias 2 -> 1
- net GND: vias 4 -> 5
Other:
- board text added: "By Ender"

Commit message: pcb terminado
Parts:
- removed C5, C6: 100nF, EESTN5:C_1206
- removed D1, D2, D3, D4, D5, D6, D7, D8: 1n4001, EESTN5:sod123
- removed J6: batt, EESTN5:BORNERA2_AZUL
- removed J8, J9: LED_izq, EESTN5:Pin_Strip_3
- removed R3: 10k, EESTN5:R_1206
- removed SW1: SW_SPDT, EESTN5:SW_SPDT_TH_Vertical
- removed U3: L7805, EESTN5:TO-220
- removed hole_2mm (x3): VAL**, EESTN5:hole_2mm
- added C10: 100nF, EESTN5:C_1206, B.Cu at (165.9, 57.8)
- added C11: 100nF, EESTN5:C_1206, B.Cu at (153.6, 65.0)
- added C12: 10uF 16v, EESTN5:CAP_ELEC_5x11mm, F.Cu at (158.7, 66.4)
- added C2: 100nF, EESTN5:C_1206, F.Cu at (158.0, 56.1)
- added C9: 100uF 25v, EESTN5:CAP_ELEC_5x11mm, F.Cu at (165.6, 62.6)
- added J11: batt, EESTN5:Pin_Header_2, F.Cu at (145.9, 71.3)
- added J3: motor dir, EESTN5:Pin_Header_2, F.Cu at (141.7, 71.2)
- added R2: 10k, EESTN5:R_1206, B.Cu at (136.6, 48.5)
- added SW2: SW_SPDT, EESTN5:Pin_Strip_3, F.Cu at (151.5, 72.5)
- added U2: TA6586, EESTN5:DIP-8, F.Cu at (130.0, 64.9)
- added U7: L7805, EESTN5:TO-220, F.Cu at (161.9, 72.4)
- C1: value 220uf -> 10uF; footprint EESTN5:CAP_ELEC_5x11mm -> EESTN5:C_1206
- C3: value 100uF 25v -> 10uF; footprint EESTN5:CAP_ELEC_5x11mm -> EESTN5:C_1206
- C4: value 10uF 16v -> 22uF 25v
- C7, C8, U5: moved to B.Cu
- J1: value motores izq -> motor izq; footprint EESTN5:JST-4V -> EESTN5:Pin_Header_2
- J2: value motores der -> motor der; footprint EESTN5:JST-4V -> EESTN5:Pin_Header_2
- J4: value esp32 usb y batt -> programmer; footprint EESTN5:Pin_Header_6 -> EESTN5:Pin_Strip_5
- U1: value L298(H)N -> TB6612FNG; footprint Package_TO_SOT_THT:TO-220-15_P2.54x2.54mm_StaggerEven_Lead4.58mm_Vertical -> Package_SO:SSOP-24_5.3x8.2mm_P0.65mm
- U4: footprint Espressif:ESP32-WROOM-32E -> esp32e:XCVR_ESP32-WROOM-32E__16MB_
- moved C4 112.8 mm to (162.9, 41.7), turned to -90 degrees
- moved C8 102.8 mm to (145.1, 55.6)
- moved C7 100.5 mm to (141.6, 44.6), turned to 180 degrees
- moved J4 97.5 mm to (159.4, 36.8), turned to 180 degrees
- moved U5 96.9 mm to (143.3, 49.9)
- moved J1 93.1 mm to (168.7, 53.0), turned to -90 degrees
- moved C3 87.9 mm to (156.7, 42.0), turned to -90 degrees
- moved J2 81.0 mm to (168.1, 47.4), turned to 90 degrees
- moved U4 79.4 mm to (142.6, 48.6)
- moved U1 77.2 mm to (160.2, 50.0), turned to 180 degrees
- moved D9 72.9 mm to (146.5, 63.9), turned to 0 degrees
- moved C1 71.5 mm to (158.0, 59.8)
- moved R1 69.2 mm to (146.2, 66.8)
Connections:
- C1 pad 1: VCC -> +5V
- C4 pad 1: +5V -> VCC
- J1 pad 1: Net-(D7-A) -> Net-(J1-Pad1)
- J1 pad 2: Net-(D1-A) -> Net-(J1-Pad2)
- J2 pad 1: Net-(D3-A) -> Net-(J2-Pad1)
- J2 pad 2: Net-(D5-A) -> Net-(J2-Pad2)
- J4 pad 1: /salida -> /rx
- J4 pad 2: +3.3V -> /tx
- J4 pad 3: /EN -> +3.3V
- J4 pad 4: /TX -> /en
- J4 pad 5: /RX -> GND
- U1 pad 1: GND -> Net-(J1-Pad2)
- U1 pad 10: /IN4 -> GND
- U1 pad 11: +5V -> Net-(J2-Pad2)
- U1 pad 12: /IN3 -> Net-(J2-Pad2)
- U1 pad 13: Net-(D7-A) -> VCC
- U1 pad 14: Net-(D5-A) -> VCC
- U1 pad 15: GND -> /PWB
- U1 pad 2: Net-(D3-A) -> Net-(J1-Pad2)
- U1 pad 3: Net-(D1-A) -> GND
- U1 pad 4: VCC -> GND
- U1 pad 5: /IN2 -> Net-(J1-Pad1)
- U1 pad 6: +5V -> Net-(J1-Pad1)
- U1 pad 7: /IN1 -> Net-(J2-Pad1)
- U1 pad 8: GND -> Net-(J2-Pad1)
- U1 pad 9: +5V -> GND
- U4 pad 10: unconnected-(U4-DAC_1/ADC2_CH8/GPIO25-Pad10) -> /buzz
- U4 pad 13: unconnected-(U4-MTMS/GPIO14/ADC2_CH6-Pad13) -> /pin_dirA
- U4 pad 16: unconnected-(U4-MTCK/GPIO13/ADC2_CH4-Pad16) -> /pin_dirB
- U4 pad 27: /Led_Izq -> /PWA
- U4 pad 28: /Led_Der -> /IN2
- U4 pad 3: /EN -> /en
- U4 pad 30: /IN2 -> /IN1
- U4 pad 31: /IN1 -> /IN3
- U4 pad 34: /RX -> /rx
- U4 pad 35: /TX -> /tx
- U4 pad 36: /IN3 -> /PWB
- U4 pad 9: unconnected-(U4-32K_XN/GPIO33/ADC1_CH5-Pad9) -> /led
Routing:
- net Net-(D5-A): track 76.5 -> 0.00 mm
- net Net-(D3-A): track 73.5 -> 0.00 mm
- net VCC: track 134.0 -> 87.6 mm, vias 0 -> 2
- net Net-(D1-A): track 45.7 -> 0.00 mm
- net /TX: track 40.1 -> 0.00 mm, vias 1 -> 0
- net Net-(D7-A): track 35.8 -> 0.00 mm
- net /en: track 0.00 -> 35.4 mm, vias 0 -> 1
- net +5V: track 108.5 -> 77.6 mm, vias 1 -> 3
- net /EN: track 27.5 -> 0.00 mm, vias 1 -> 0
- net /Led_Der: track 25.6 -> 0.00 mm, vias 1 -> 0
- net /rx: track 0.00 -> 25.1 mm, vias 0 -> 1
- net /RX: track 22.9 -> 0.00 mm, vias 1 -> 0
- net /salida: track 20.7 -> 0.00 mm
- net /IN4: track 26.3 -> 5.85 mm
- net /tx: track 0.00 -> 18.4 mm, vias 0 -> 1
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Other:
- board size 55 x 48 mm -> 45 x 45 mm
- board text removed: "By Ender"
