File: LightNing 3.0.kicad_sch (KiCad schematic)
At the start: 35 parts, among them J1 Motor_Izq_B, J2 Motor_Der_A, J3 Motor_Izq_A, J4 Motor_Der_B, J5 Jack DC, J6 batt, J7 salida esp-usb, J8 LED_izq, J9 LED_izq, SW1 SW_SPDT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

Commit message: uno cambio lokos
Parts:
- removed C2: 100uF 25v, EESTN5:CAP_ELEC_SMD_4X5.5, symbol EESTN5:CAPAPOL
- removed J1: Motor_Izq_B, EESTN5:BORNERA2_AZUL, symbol EESTN5:TB_1X2
- removed J2: Motor_Der_A, EESTN5:BORNERA2_AZUL, symbol EESTN5:TB_1X2
- removed J3: Motor_Izq_A, EESTN5:BORNERA2_AZUL, symbol EESTN5:TB_1X2
- removed J4: Motor_Der_B, EESTN5:BORNERA2_AZUL, symbol EESTN5:TB_1X2
- removed J5: Jack DC, Connector_BarrelJack:BarrelJack_Kycon_KLDX-0202-xC_Horizontal, symbol Connector:Barrel_Jack_Switch
- removed J7: salida esp-usb, EESTN5:Pin_Header_5, symbol Connector_Generic:Conn_01x05
- removed R2: 22 2W, EESTN5:RES0.3, symbol EESTN5:R
- removed U2: L7805, EESTN5:TO-220, symbol Regulator_Linear:L7805
- added J1: motores izq, EESTN5:JST-4V, symbol Connector_Generic:Conn_01x04
- added J2: motores der, EESTN5:JST-4V, symbol Connector_Generic:Conn_01x04
- added J4: esp32 usb y batt, EESTN5:Pin_Header_6, symbol Connector_Generic:Conn_01x06
- C1, C3, C4: footprint EESTN5:CAP_ELEC_SMD_4X5.5 -> EESTN5:CAP_ELEC_5x11mm
- D9: footprint LED_SMD:LED_0603_1608Metric_Pad1.05x0.95mm_HandSolder -> EESTN5:LED_1206
- J8, J9: footprint EESTN5:JST-3V -> EESTN5:Pin_Strip_3
- R1: value 330 -> 220
Connections:
- net +3.3V: now also J4.2 (Pin_2); no longer J8.1 (Pin_1), J9.1 (Pin_1)
- net +5V: now also J8.1 (Pin_1), J9.1 (Pin_1)
- net EN: now also J4.3 (Pin_3)
- net GND: now also R1.2, J4.6 (Pin_6)
- net IN1: now also U1.7 (IN2); no longer U1.5 (IN1)
- net IN2: now also U1.5 (IN1); no longer U1.7 (IN2)
- net IN3: now also U1.12 (IN4); no longer U1.10 (IN3)
- net IN4: now also U1.10 (IN3); no longer U1.12 (IN4)
- net Led_Der: now also U4.28 (GPIO17); no longer U4.11 (DAC_2/ADC2_CH9/GPIO26)
- net Led_Izq: now also U4.27 (GPIO16); no longer U4.10 (DAC_1/ADC2_CH8/GPIO25)
- net RX: now also J4.5 (Pin_5)
- net TX: now also J4.4 (Pin_4)
- net at D9.1 (K): now also R1.1; no longer SW1.1 (A)
- net at D7.1 (A), D8.2 (K), U1.13 (OUT3): now also J1.1 (Pin_1), J1.4 (Pin_4)
- net at D5.1 (A), D6.2 (K), U1.14 (OUT4): now also J2.2 (Pin_2), J2.3 (Pin_3)
- net at D3.1 (A), D4.2 (K), U1.2 (OUT1): now also J2.1 (Pin_1), J2.4 (Pin_4)
- net at D1.1 (A), D2.2 (K), U1.3 (OUT2): now also J1.2 (Pin_2), J1.3 (Pin_3)
- net at D9.2 (A): now also U4.24 (ADC2_CH2/GPIO2); no longer R1.2
- new net salida: J4.1 (Pin_1), SW1.1 (A)
Other:
- note removed: "cargador"
- moved on the sheet: C3, C4, C5, C6, J6, J8, J9, SW1, U3

Commit message: rework
Parts:
- removed C3: 100uF 25v, EESTN5:CAP_ELEC_5x11mm, symbol EESTN5:CAPAPOL
- removed C4: 10uF 16v, EESTN5:CAP_ELEC_5x11mm, symbol EESTN5:CAPAPOL
- removed C5, C6: 100nF, EESTN5:C_1206, symbol EESTN5:C
- removed J4: esp32 usb y batt, EESTN5:Pin_Header_6, symbol Connector_Generic:Conn_01x06
- removed J6: batt, EESTN5:BORNERA2_AZUL, symbol EESTN5:TB_1X2
- removed J9: LED_izq, EESTN5:Pin_Strip_3, symbol Connector_Generic:Conn_01x03
- removed R3: 10k, EESTN5:R_1206, symbol EESTN5:R
- added C2: 100uF 25v, EESTN5:CAP_ELEC_5x11mm, symbol EESTN5:CAPAPOL
- added C3, C4: 100nF, EESTN5:CAP_0.1, symbol EESTN5:C
- added C5: 10uF 16v, EESTN5:CAP_ELEC_5x11mm, symbol EESTN5:CAPAPOL
- added J3: batt, EESTN5:Pin_Header_2, symbol EESTN5:TB_1X2
- added J4: LED_izq, EESTN5:Pin_Strip_3, symbol Connector_Generic:Conn_01x03
- added J5: salida a modulo, EESTN5:pin_strip_4, symbol Connector_Generic:Conn_01x04
- added J6: Sharp A, EESTN5:Pin_Strip_3, symbol Connector_Generic:Conn_01x03
- added J7: Sharp B, EESTN5:Pin_Strip_3, symbol Connector_Generic:Conn_01x03
- added R2: 10k, EESTN5:R_1206, symbol EESTN5:R
- D1, D2, D3, D4, D5, D6, D7, D8: footprint EESTN5:sod123 -> EESTN5:DO-41
- J1, J2: footprint EESTN5:JST-4V -> EESTN5:pin_strip_4
- J8: value LED_izq -> ampBuzz
- SW1: footprint EESTN5:SW_SPDT_TH_Vertical -> EESTN5:Pin_Strip_3
Connections:
- net Led_Der is gone; now on net IN2: U4.28 (GPIO17)
- net +3.3V: now also R2.1
- net +5V: now also C4.1, C5.1, J4.1 (Pin_1), J5.3 (Pin_3), J6.2 (Pin_2), J7.2 (Pin_2)
- net EN: now also R2.2; no longer U4.3 (EN/CHIP_PU)
- net GND: now also C2.2, C3.2, C4.2, C5.2, J3.2, J4.3 (Pin_3), J5.1 (Pin_1), J6.3 (Pin_3), J7.3 (Pin_3)
- net IN1: now also U1.5 (IN1), U4.27 (GPIO16); no longer U1.7 (IN2), U4.31 (GPIO19)
- net IN2: now also U1.7 (IN2); no longer U1.5 (IN1), U4.30 (GPIO18)
- net IN3: now also U1.10 (IN3), U4.30 (GPIO18); no longer U1.12 (IN4), U4.36 (GPIO22)
- net IN4: now also U1.12 (IN4), U4.31 (GPIO19); no longer U1.10 (IN3), U4.33 (GPIO21)
- net VCC: now also C2.1, C3.1, J5.4 (Pin_4)
- net at D3.1 (A), D4.2 (K), U1.2 (OUT1): now also J1.1 (Pin_1), J1.4 (Pin_4); no longer J2.1 (Pin_1), J2.4 (Pin_4)
- net at SW1.2 (B): now also J3.1
- net at D7.1 (A), D8.2 (K), U1.13 (OUT3): now also J2.1 (Pin_1), J2.4 (Pin_4); no longer J1.1 (Pin_1), J1.4 (Pin_4)
- net buzz: now reaches U4.10 (DAC_1/ADC2_CH8/GPIO25)
- net buzz: now also J8.2 (Pin_2)
- net sensor_b: now reaches U4.13 (MTMS/GPIO14/ADC2_CH6)
- net sensor_b: now also J7.1 (Pin_1)
- net sensor_a: now reaches U4.16 (MTCK/GPIO13/ADC2_CH4)
- net sensor_a: now also J6.1 (Pin_1)
- net led: now reaches U4.9 (32K_XN/GPIO33/ADC1_CH5)
- net led: now also J4.2 (Pin_2)
- removed net Led_Izq: J8.2 (Pin_2), U4.27 (GPIO16)
- net RX: no longer names the net of U4.34 (U0RXD/GPIO3)
- net TX: no longer names the net of U4.35 (U0TXD/GPIO1)
- net salida renamed Cargador
- net Cargador: now also J5.2 (Pin_2)
Other:
- note added: "SALIDA A MODULO BATERIA"
- note added: "buzzer"
- note added: "sensores SHARP"
- note removed: "salida ESp32 a modulo usb"

Commit message: pcb terminado
Parts:
- removed C1: 220uf, EESTN5:CAP_ELEC_5x11mm, symbol StepperDriver-rescue:CP_Small-Device
- removed D1, D2, D3, D4, D5, D6, D7, D8: 1n4001, EESTN5:DO-41, symbol EESTN5:DIODE
- removed J1: motores izq, EESTN5:pin_strip_4, symbol Connector_Generic:Conn_01x04
- removed J2: motores der, EESTN5:pin_strip_4, symbol Connector_Generic:Conn_01x04
- removed J4: LED_izq, EESTN5:Pin_Strip_3, symbol Connector_Generic:Conn_01x03
- removed J5: salida a modulo, EESTN5:pin_strip_4, symbol Connector_Generic:Conn_01x04
- removed J6: Sharp A, EESTN5:Pin_Strip_3, symbol Connector_Generic:Conn_01x03
- removed J7: Sharp B, EESTN5:Pin_Strip_3, symbol Connector_Generic:Conn_01x03
- removed J8: ampBuzz, EESTN5:Pin_Strip_3, symbol Connector_Generic:Conn_01x03
- removed U1: L298(H)N, Package_TO_SOT_THT:TO-220-15_P2.54x2.54mm_StaggerEven_Lead4.58mm_Vertical, symbol EESTN5:L298(H)N
- added C2: 22uF 25v, EESTN5:CAP_ELEC_5x11mm, symbol EESTN5:CAPAPOL
- added C3 (x2): 10uF, EESTN5:C_1206, symbol EESTN5:C
- added C3: 100nF, EESTN5:C_1206, symbol EESTN5:C
- added J1: motor izq, EESTN5:Pin_Header_2, symbol EESTN5:TB_1X2
- added J2: motor der, EESTN5:Pin_Header_2, symbol EESTN5:TB_1X2
- added J3: motor dir, EESTN5:Pin_Header_2, symbol EESTN5:TB_1X2
- added J4: programmer, EESTN5:Pin_Strip_5, symbol Connector_Generic:Conn_01x05
- added U1: TB6612FNG, Package_SO:SSOP-24_5.3x8.2mm_P0.65mm, symbol Driver_Motor:TB6612FNG
- added U2: TA6586, EESTN5:DIP-8, symbol Driver_FET:FAN3278
- C3, C4: footprint EESTN5:CAP_0.1 -> EESTN5:C_1206
- U4: footprint Espressif:ESP32-WROOM-32E -> esp32e:XCVR_ESP32-WROOM-32E__16MB_
Connections:
- net EN is gone; now on net en: R2.2
- net +3.3V: now also J4.3 (Pin_3)
- net +5V: now also C3.1, C3.1, U1.19 (STBY), U1.20 (VCC)
- net GND: now also C2.2, C3.2, C3.2, C3.2, J4.5 (Pin_5), U1.10 (PGND2), U1.18 (GND), U1.3 (PGND1), U1.4 (PGND1), U1.9 (PGND2), U2.3 (GND)
- net IN1: now also U4.30 (GPIO18), U1.21 (AIN1); no longer U4.27 (GPIO16)
- net IN2: now also U1.22 (AIN2)
- net IN3: now also U4.31 (GPIO19), U1.17 (BIN1); no longer U4.30 (GPIO18)
- net IN4: now also U4.33 (GPIO21), U1.16 (BIN2); no longer U4.31 (GPIO19)
- net VCC: now also C2.1, C3.1, U1.13 (VM2), U1.14 (VM3), U1.24 (VM1), U2.4 (VCC)
- net en: now reaches U4.3 (EN/CHIP_PU)
- net en: now also J4.4 (Pin_4)
- net rx: now reaches U4.34 (U0RXD/GPIO3)
- net rx: now also J4.1 (Pin_1)
- net tx: now reaches U4.35 (U0TXD/GPIO1)
- net tx: now also J4.2 (Pin_2)
- net PWB: now reaches U4.36 (GPIO22)
- net PWB: now also U1.15 (PWMB)
- net Cargador: no longer names the net of SW1.1 (A)
- net sensor_a renamed pin_dirB
- net pin_dirB: now also U2.1 (BI)
- net sensor_b renamed pin_dirA
- net pin_dirA: now also U2.2 (FI)
- new net: J3.1, U2.5 (FO), U2.6 (FO)
- new net: J3.2, U2.7 (BO), U2.8 (BO)
- new net: J2.1, U1.7 (BO2), U1.8 (BO2)
- new net: J2.2, U1.11 (BO1), U1.12 (BO1)
- new net: J1.2, U1.1 (AO1), U1.2 (AO1)
- new net: J1.1, U1.5 (AO2), U1.6 (AO2)
- new net PWA: U1.23 (PWMA), U4.27 (GPIO16)
- no-connect marks 0 -> 1
Other:
- note added: "DRIVER TB6612"
- note added: "drv ta6586"
- note added: "programmer"
- note removed: "DRIVER L298N"
- note removed: "Leds rgb"
- note removed: "SALIDA A MODULO BATERIA"
- note removed: "buzzer"
- note removed: "sensores SHARP"
- moved on the sheet: C2, C3, C4, C5, C7, C8, D9, J3, R1, R2, SW1, U3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
