File: LightNing 3.0 PCB/LightNing 3.0.kicad_pcb (KiCad board)
At the start: 2 copper layers, 45 x 45 mm, 24 parts, among them J1 motor izq, J11 batt, J2 motor der, J3 motor dir, J4 programmer, SW2 SW_SPDT, U1 TB6612FNG, U2 TA6586, U4 ESP32-WROOM-E, U5 AMS1117-3.3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

Commit message: update 1 november
Parts:
- added hole_2mm: VAL**, EESTN5:hole_2mm, F.Cu at (127.5, 77.5)
- added hole_2mm: VAL**, EESTN5:hole_2mm, F.Cu at (167.5, 77.5)
- added hole_2mm: VAL**, EESTN5:hole_2mm, F.Cu at (127.5, 37.5)
